Commit message: Add my file

File: kinova_description/urdf/j2n6s300.xacro (robot description, xacro)
@@ -94,5 +94,5 @@
     <xacro:property name="joint_6_origin_rpy" value="${J_PI/3} 0 ${J_PI}" />
     <!-- If gripper inverted, use this line instead -->
-    <!-- <xacro:property name="joint_6_origin_rpy" value="$${-J_PI/3} 0 0" /> -->
+     <!-- <xacro:property name="joint_6_origin_rpy" value="${-J_PI/3} 0 0" />  -->
     <xacro:property name="joint_6_lower_limit" value="${-2*J_PI}" />
     <xacro:property name="joint_6_upper_limit" value="${2*J_PI}" />
